File: classic/bluepill.sch (KiCad schematic (older format))
At the start: 37 parts, among them J1 USB_B_Micro, J2 Boot, J3 Left Row, J4 Right Row, J5 SWD, SW1 Reset, U1 RT8183-33, U2 STM32F103C8Tx, Y1 8MHz, Y2 32768Hz

Commit message: references
Parts:
- removed C11: 100n, Capacitor_SMD:C_0603_1608Metric_Pad1.05x0.95mm_HandSolder, symbol Device:C
- removed D4: BAT60J, Diode_SMD:D_SOD-323_HandSoldering, symbol Diode:1N5819
- C1: footprint Capacitor_SMD:C_0603_1608Metric_Pad1.05x0.95mm_HandSolder -> Capacitor_SMD:C_0805_2012Metric_Pad1.15x1.40mm_HandSolder
- C4: renamed from C3; footprint Capacitor_SMD:C_0603_1608Metric_Pad1.05x0.95mm_HandSolder -> Capacitor_SMD:C_0805_2012Metric_Pad1.15x1.40mm_HandSolder
- gave numbers to parts that had none: 1
- renumbered C9 to C10, C10 to C11, C2 to C3, C4 to C5, C5 to C6, C6 to C7, C7 to C8, C8 to C9, D2 to D1, D3 to D2, R5 to R4, R4 to R5
Connections:
- net +3V3: now also J5.4 (Pin_4); no longer J5.1 (Pin_1)
- net GNDREF: now also J5.1 (Pin_1); no longer J5.4 (Pin_4)
- net SWCLK: now also J5.2 (Pin_2); no longer J5.3 (Pin_3)
- net SWDIO: now also J5.3 (Pin_3); no longer J5.2 (Pin_2)
Other:
- note added: "BluePill boards from TaoBao have diferent design:\n+ extra 1M or 10M resistor between OSCIN | OSCOUT \n- no GND connection for capacitors\nSame concept can be found on some RedPill boards.\nRecommended design from STM has no resistor!\nIn this schematic it is OPTIONAL!\nBluePill uses crystal in HC-49S (HC-49-4H) package.\nBlackPill uses both: resistor (10M) and \ngrounding for capacitors."
- note added: "Not Present on original BluePill.\nHighly recomended.\n\nPass the 3V3 and Vbat from header through\nseparate (individual) diodes.\nMerge behind diodes, decouple with 100nF.\nProvide this to Vbat of microcontroller."
- note added: "Typically used diodes:\n- 1N5819: in SOD123F or DO-41\n- LSM115JE3/TR13 : DO-214BA\n- BAS70 : in SOT23\n- 1N4448 : in SOD123"
- note removed: "BluePill boards from TaoBao have diferent design:\n+ extra 1M or 10M resistor between OSCIN | OSCOUT \n- no GND connection for capacitors\nSame concept can be found on some RedPill boards.\nRecommended design from STM has no resistor!\nIn this schematic it is OPTIONAL!\nBluePill uses crystal in HC-49S (HC-49-4H) package.\nBlackPill uses both: resistor (10M) and grounding."
- note removed: "Not Present on original BluePill.\nHighly recomended.\nCan be done with:\n- 1N5819: in SOD123F or DO-41\n- LSM115JE3/TR13 : DO-214BA\n- BAS70 : in SOT23\n- 1N4448 : in SOD123"
