File: reforged/bluepill_reforged.kicad_pcb (KiCad board)
At the start: 2 copper layers, 22.9 x 53.3 mm, 35 parts, among them J1 USB_B_Micro, J2 Boot, J3 Left Row, J4 Right Row, J5 SWD, SW1 Reset, U1 RT8183-33, U2 STM32F103C8Tx, Y1 8MHz, Y2 32768Hz

Commit message: references
Parts:
- removed C14: 100n, Capacitor_SMD:C_0603_1608Metric_Pad1.05x0.95mm_HandSolder
- removed J5: SWD, Connector_PinHeader_2.54mm:PinHeader_1x04_P2.54mm_Horizontal
- added D3: Power, LED_SMD:LED_0805_2012Metric_Castellated, F.Cu at (116.5, 95.9)
- added D4: 1N5819, Diode_THT:D_DO-41_SOD81_P10.16mm_Horizontal, F.Cu at (168.1, 60.2)
- added D5: 1N5819, Diode_THT:D_DO-41_SOD81_P10.16mm_Horizontal, F.Cu at (154.2, 60.2)
- added R10: 510, Resistor_SMD:R_0603_1608Metric_Pad1.05x0.95mm_HandSolder, F.Cu at (126.8, 95.9)
- added R11: 510, Resistor_SMD:R_0603_1608Metric_Pad1.05x0.95mm_HandSolder, F.Cu at (98.2, 96.5)
- added SW2: Reset, Button_Switch_SMD:SW_SPST_B3U-1000P, F.Cu at (110.5, 63.9)
- C1: value 1u -> 0.1-10 uF; footprint Capacitor_SMD:C_0805_2012Metric_Pad1.15x1.40mm_HandSolder -> Capacitor_Tantalum_SMD:CP_EIA-6032-20_AVX-F_Pad2.25x2.35mm_HandSolder; moved to F.Cu
- C2: value 100n -> 47-1000 uF; footprint Capacitor_SMD:C_0603_1608Metric_Pad1.05x0.95mm_HandSolder -> Capacitor_Tantalum_SMD:CP_EIA-6032-20_AVX-F_Pad2.25x2.35mm_HandSolder; moved to F.Cu
- C3: value 22n -> 1uF; moved to F.Cu
- C4: value 1u -> 20pF; footprint Capacitor_SMD:C_0805_2012Metric_Pad1.15x1.40mm_HandSolder -> Capacitor_SMD:C_0603_1608Metric_Pad1.05x0.95mm_HandSolder
- C5, C6, C7: moved to B.Cu
- C8: value 20pF -> 1uF
- C9: value 100nF -> 100n
- D1: value PC13 -> Protection; footprint LED_SMD:LED_0603_1608Metric_Pad1.05x0.95mm_HandSolder -> Diode_SMD:D_SMA_Handsoldering
- D2: value PWR -> Green; footprint LED_SMD:LED_0603_1608Metric_Pad1.05x0.95mm_HandSolder -> LED_SMD:LED_0805_2012Metric_Castellated
- J1: value USB_B_Micro -> USB_C_Receptacle_USB2.0; footprint Connector_USB:USB_Micro-B_Wuerth_629105150521 -> Connector_USB:USB_C_Receptacle_Palconn_UTC16-G
- J2: value Boot -> Left Castellation; footprint Connector_PinHeader_2.54mm:PinHeader_2x03_P2.54mm_Vertical -> Connector_PinHeader_2.54mm:PinHeader_1x20_P2.54mm_Vertical; moved to B.Cu
- J3: value Left Row -> Cortex debug; footprint Connector_PinHeader_2.54mm:PinHeader_1x20_P2.54mm_Vertical -> Connector_PinHeader_1.27mm:PinHeader_2x05_P1.27mm_Vertical_SMD; moved to F.Cu
- J4: value Right Row -> Right Castellation
- R1: value 100K -> 5K1; moved to B.Cu
- R2: value 22R -> 5K1; moved to B.Cu
- R4: value 1.5K -> 100K
- R5: value 100K -> 10K
- R6: value 10M [N/A] -> 22R; moved to F.Cu
- R7: value 10K -> 1.5K
- R8: value 510 -> 10M [N/A]; moved to B.Cu
- R9: value 510 -> 10K
- SW1: value Reset -> Boot0; footprint Button_Switch_SMD:SW_SPST_TL3342 -> Button_Switch_SMD:SW_SPST_B3U-1000P
- U1: value RT8183-33 -> AMS1117-3.3; footprint Package_TO_SOT_SMD:SOT-353_SC-70-5_Handsoldering -> Package_TO_SOT_SMD:SOT-223-3_TabPin2; moved to F.Cu
- moved C2 93.5 mm to (178.0, 75.9), turned to 0 degrees
- moved U1 84.5 mm to (168.6, 71.0), turned to 0 degrees
- moved C3 81.5 mm to (163.2, 91.2), turned to 0 degrees
- moved C1 75.6 mm to (156.8, 80.6)
- moved D1 61.5 mm to (130.8, 55.1), turned to 0 degrees
- moved C8 58.7 mm to (163.2, 88.7)
- moved C9 58.4 mm to (167.6, 86.2)
- moved C12 53.8 mm to (158.9, 86.8)
- moved C11 51.4 mm to (163.2, 93.7)
- moved C10 49.3 mm to (163.2, 86.2)
- moved C13 49.3 mm to (158.9, 84.3)
- moved R6 45.1 mm to (129.5, 69.6)
- moved J2 43.6 mm to (105.4, 101.6)
- moved R2 37.4 mm to (111.1, 53.3), turned to 180 degrees
- moved C4 34.9 mm to (113.0, 85.7), turned to 0 degrees
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Connections:
- C1 pad 1: GNDREF -> +5V
- C1 pad 2: +5V -> GNDREF
- C10 pad 1: GNDREF -> +3V3
- C10 pad 2: +3V3 -> GNDREF
- C2 pad 1: +5V -> +3V3
- C3 pad 1: GNDREF -> BOOT0
- C3 pad 2: Net-(C3-Pad2) -> GNDREF
- C4 pad 1: GNDREF -> OSCIN
- C4 pad 2: +3V3 -> GNDREF
- C5 pad 1: OSCIN -> PC14
- C6 pad 1: PC14 -> OSCOUT
- C7 pad 1: OSCOUT -> PC15
- C8 pad 1: PC15 -> NRST
- C9 pad 1: NRST -> VBAT_Protected
- D1 pad 1: Net-(D1-Pad1) -> +5V
- D1 pad 2: +3V3 -> VBUS
- J2 pad 2: +3V3 -> GNDREF
- J2 pad 3: Net-(J2-Pad3) -> +5V
- J2 pad 4: Net-(J2-Pad4) -> PB9
- J2 pad 5: GNDREF -> PB8
- J2 pad 6: GNDREF -> PB7
- J3 pad 10: PB3 -> NRST
- J3 pad 2: GNDREF -> PA13
- J3 pad 3: +5V -> GNDREF
- J3 pad 4: PB9 -> PA14
- J3 pad 5: PB8 -> GNDREF
- J3 pad 6: PB7 -> PB3
- J3 pad 7: PB6 -> Net-(J3-Pad7)
- J3 pad 8: PB5 -> Net-(J3-Pad8)
- J3 pad 9: PB4 -> GNDREF
- R1 pad 1: BOOT0 -> Net-(J1-PadA5)
- R1 pad 2: Net-(J2-Pad3) -> GNDREF
- R2 pad 1: D- -> Net-(J1-PadB5)
- R2 pad 2: PA11 -> GNDREF
- R3 pad 1: PA12 -> D-
- R3 pad 2: D+ -> PA11
- R4 pad 1: +3V3 -> GNDREF
- R4 pad 2: PA12 -> BOOT0
- R5 pad 1: Net-(J2-Pad4) -> GNDREF
- R6 pad 1: OSCIN -> PA12
- R6 pad 2: OSCOUT -> D+
- R7 pad 1: NRST -> +3V3
- R7 pad 2: +3V3 -> PA12
- R8 pad 1: PC13 -> OSCIN
- R8 pad 2: Net-(D1-Pad1) -> OSCOUT
- R9 pad 1: GNDREF -> NRST
- R9 pad 2: Net-(D2-Pad1) -> +3V3
- SW1 pad 1: GNDREF -> +3V3
- SW1 pad 2: NRST -> BOOT0
- U1 pad 1: +5V -> GNDREF
- U1 pad 2: GNDREF -> +3V3
- U2 pad 1: +BATT -> VBAT_Protected
- U2 pad 34: SWDIO -> PA13
- U2 pad 37: SWCLK -> PA14
