File: project files/classic/bluepill.sch (KiCad schematic (older format))
At the start: 38 parts, among them J1 USB_B_Micro, J2 Boot, J3 Left Row, J4 Right Row, J5 SWD, SW1 Reset, U1 RT8183-33, U2 STM32F103C8Tx, Y1 8MHz, Y2 32768Hz

Commit message: Update bluepill.sch
Other:
- note added: "Another suggestion is to use polymer resettable fuse like:\n- case 1210 (inch) : from Samsung Tab batteries\n- case 1206 : typically used on ST-Link clones"
- note added: "Originally, BluePill contained RT8183-B as voltage regulator. It is outdated. \nDirect replacement: RT9193-33GB, but it is capable to deliver up to 300mA.\nBoth seems to be a copy of LDK-130-3.3 in SOT23-5 (SOT323-5L) package.\nPinout compatible with:\n- AP2210-3.3 : up to 300 mA\n"
- note added: "Some clones uses AMS1117 as Linear Voltage Regulator\nwith tantalum SMD capacitors:\n- Pre-capacitor: 7343 Metric Package : \n- Post-capacitor: 7343 Metric Package :"
- note removed: "Originally, BluePill contained RT8183-B as voltage regulator. It is outdated. \nDirect replacement: RT9193-33GB, but it is capable to deliver up to 300mA.\nBoth seems to be a copy of LDK-130-3.3 in SOT23-5 (SOT323-5L) package.\n"
- note removed: "Some clones uses AMS1117 as Linear Voltage Regulator\nwith tantalum SMD capacitors:\n- Pre-capacitor\n- Post-capacitor"
- moved on the sheet: C1, C3, C4, U1
Changed lines of the file:
@@
 L power:+3.3V #PWR09
 U 1 1 5E0C47D9
-P 2800 5300
-F 0 "#PWR09" H 2800 5150 50  0001 C CNN
-F 1 "+3.3V" H 2815 5473 50  0000 C CNN
-F 2 "" H 2800 5300 50  0001 C CNN
-F 3 "" H 2800 5300 50  0001 C CNN
-	1    2800 5300
+P 2850 5650
+F 0 "#PWR09" H 2850 5500 50  0001 C CNN
+F 1 "+3.3V" H 2865 5823 50  0000 C CNN
+F 2 "" H 2850 5650 50  0001 C CNN
+F 3 "" H 2850 5650 50  0001 C CNN
+	1    2850 5650
 	1    0    0    -1
 $EndComp
@@
 L power:+5V #PWR02
 U 1 1 5E0CACD2
-P 1600 5300
-F 0 "#PWR02" H 1600 5150 50  0001 C CNN
-F 1 "+5V" H 1615 5473 50  0000 C CNN
-F 2 "" H 1600 5300 50  0001 C CNN
-F 3 "" H 1600 5300 50  0001 C CNN
-	1    1600 5300
+P 1650 5650
+F 0 "#PWR02" H 1650 5500 50  0001 C CNN
+F 1 "+5V" H 1665 5823 50  0000 C CNN
+F 2 "" H 1650 5650 50  0001 C CNN
+F 3 "" H 1650 5650 50  0001 C CNN
+	1    1650 5650
 	1    0    0    -1
 $EndComp
@@
 Power Supply
 Text Notes 600  4950 0    50   ~ 0
-Originally, BluePill contained RT8183-B as voltage regulator. It is outdated. \nDirect replacement: RT9193-33GB, but it is capable to deliver up to 300mA.\nBoth seems to be a copy of LDK-130-3.3 in SOT23-5 (SOT323-5L) package.\n
+Originally, BluePill contained RT8183-B as voltage regulator. It is outdated. \nDirect replacement: RT9193-33GB, but it is capable to deliver up to 300mA.\nBoth seems to be a copy of LDK-130-3.3 in SOT23-5 (SOT323-5L) package.\nPinout compatible with:\n- AP2210-3.3 : up to 300 mA\n
 $Comp
 L Regulator_Linear:LDK130-33_SOT23_SOT353 U1
 U 1 1 5E1140B5
-P 2050 5500
-F 0 "U1" H 2050 5842 50  0000 C CNN
-F 1 "RT8183-33" H 2050 5751 50  0000 C CNN
-F 2 "Package_TO_SOT_SMD:SOT-353_SC-70-5_Handsoldering" H 2050 5825 50  0001 C CNN
-F 3 "http://www.st.com/content/ccc/resource/technical/document/datasheet/29/10/f7/87/2f/66/47/f4/DM00076097.pdf/files/DM00076097.pdf/jcr:content/translations/en.DM00076097.pdf" H 2050 5500 50  0001 C CNN
-	1    2050 5500
+P 2100 5850
+F 0 "U1" H 2100 6192 50  0000 C CNN
+F 1 "RT8183-33" H 2100 6101 50  0000 C CNN
+F 2 "Package_TO_SOT_SMD:SOT-353_SC-70-5_Handsoldering" H 2100 6175 50  0001 C CNN
+F 3 "http://www.st.com/content/ccc/resource/technical/document/datasheet/29/10/f7/87/2f/66/47/f4/DM00076097.pdf/files/DM00076097.pdf/jcr:content/translations/en.DM00076097.pdf" H 2100 5850 50  0001 C CNN
+	1    2100 5850
 	1    0    0    -1
 $EndComp
@@
 L Device:C C3
 U 1 1 5E1166B3
-P 2350 5700
-F 0 "C3" H 2235 5654 50  0000 R CNN
-F 1 "22n" H 2235 5745 50  0000 R CNN
-F 2 "Capacitor_SMD:C_0603_1608Metric_Pad1.05x0.95mm_HandSolder" H 2388 5550 50  0001 C CNN
-F 3 "~" H 2350 5700 50  0001 C CNN
-	1    2350 5700
+P 2400 6050
+F 0 "C3" H 2285 6004 50  0000 R CNN
+F 1 "22n" H 2285 6095 50  0000 R CNN
+F 2 "Capacitor_SMD:C_0603_1608Metric_Pad1.05x0.95mm_HandSolder" H 2438 5900 50  0001 C CNN
+F 3 "~" H 2400 6050 50  0001 C CNN
+	1    2400 6050
 	-1   0    0    1
 $EndComp
@@
 L power:GNDREF #PWR010
 U 1 1 5E116D65
-P 2800 5850
-F 0 "#PWR010" H 2800 5600 50  0001 C CNN
-F 1 "GNDREF" H 2805 5677 50  0000 C CNN
-F 2 "" H 2800 5850 50  0001 C CNN
-F 3 "" H 2800 5850 50  0001 C CNN
-	1    2800 5850
+P 2850 6200
+F 0 "#PWR010" H 2850 5950 50  0001 C CNN
+F 1 "GNDREF" H 2855 6027 50  0000 C CNN
+F 2 "" H 2850 6200 50  0001 C CNN
+F 3 "" H 2850 6200 50  0001 C CNN
+	1    2850 6200
 	1    0    0    -1
 $EndComp
@@
 L power:GNDREF #PWR07
 U 1 1 5E117AC1
-P 2050 5850
-F 0 "#PWR07" H 2050 5600 50  0001 C CNN
-F 1 "GNDREF" H 2055 5677 50  0000 C CNN
-F 2 "" H 2050 5850 50  0001 C CNN
-F 3 "" H 2050 5850 50  0001 C CNN
-	1    2050 5850
+P 2100 6200
+F 0 "#PWR07" H 2100 5950 50  0001 C CNN
+F 1 "GNDREF" H 2105 6027 50  0000 C CNN
+F 2 "" H 2100 6200 50  0001 C CNN
+F 3 "" H 2100 6200 50  0001 C CNN
+	1    2100 6200
 	1    0    0    -1
 $EndComp
@@
 L Device:C C1
 U 1 1 5E119CEC
-P 1600 5700
-F 0 "C1" H 1485 5654 50  0000 R CNN
-F 1 "1u" H 1485 5745 50  0000 R CNN
-F 2 "Capacitor_SMD:C_0805_2012Metric_Pad1.15x1.40mm_HandSolder" H 1638 5550 50  0001 C CNN
-F 3 "~" H 1600 5700 50  0001 C CNN
-	1    1600 5700
+P 1650 6050
+F 0 "C1" H 1535 6004 50  0000 R CNN
+F 1 "1u" H 1535 6095 50  0000 R CNN
+F 2 "Capacitor_SMD:C_0805_2012Metric_Pad1.15x1.40mm_HandSolder" H 1688 5900 50  0001 C CNN
+F 3 "~" H 1650 6050 50  0001 C CNN
+	1    1650 6050
 	-1   0    0    1
 $EndComp
@@
 L power:GNDREF #PWR03
 U 1 1 5E11B4BE
-P 1600 5850
-F 0 "#PWR03" H 1600 5600 50  0001 C CNN
-F 1 "GNDREF" H 1605 5677 50  0000 C CNN
-F 2 "" H 1600 5850 50  0001 C CNN
-F 3 "" H 1600 5850 50  0001 C CNN
-	1    1600 5850
-	1    0    0    -1
-$EndComp
-Wire Wire Line
-	1750 5400 1700 5400
-Wire Wire Line
-	1600 5400 1600 5300
-Wire Wire Line
-	1600 5550 1600 5400
-Wire Wire Line
-	1750 5500 1700 5500
-Wire Wire Line
-	1700 5500 1700 5400
-Connection ~ 1700 5400
-Wire Wire Line
-	1700 5400 1600 5400
+P 1650 6200
+F 0 "#PWR03" H 1650 5950 50  0001 C CNN
+F 1 "GNDREF" H 1655 6027 50  0000 C CNN
+F 2 "" H 1650 6200 50  0001 C CNN
+F 3 "" H 1650 6200 50  0001 C CNN
+	1    1650 6200
+	1    0    0    -1
+$EndComp
+Wire Wire Line
+	1800 5750 1750 5750
+Wire Wire Line
+	1650 5750 1650 5650
+Wire Wire Line
+	1650 5900 1650 5750
+Wire Wire Line
+	1800 5850 1750 5850
+Wire Wire Line
+	1750 5850 1750 5750
+Connection ~ 1750 5750
+Wire Wire Line
+	1750 5750 1650 5750
 $Comp
 L power:GNDREF #PWR08
 U 1 1 5E133A88
-P 2350 5850
-F 0 "#PWR08" H 2350 5600 50  0001 C CNN
-F 1 "GNDREF" H 2355 5677 50  0000 C CNN
-F 2 "" H 2350 5850 50  0001 C CNN
-F 3 "" H 2350 5850 50  0001 C CNN
-	1    2350 5850
+P 2400 6200
+F 0 "#PWR08" H 2400 5950 50  0001 C CNN
+F 1 "GNDREF" H 2405 6027 50  0000 C CNN
+F 2 "" H 2400 6200 50  0001 C CNN
+F 3 "" H 2400 6200 50  0001 C CNN
+	1    2400 6200
 	1    0    0    -1
 $EndComp
@@
 L Device:C C4
 U 1 1 5E133F34
-P 2800 5700
-F 0 "C4" H 2685 5654 50  0000 R CNN
-F 1 "1u" H 2685 5745 50  0000 R CNN
-F 2 "Capacitor_SMD:C_0805_2012Metric_Pad1.15x1.40mm_HandSolder" H 2838 5550 50  0001 C CNN
-F 3 "~" H 2800 5700 50  0001 C CNN
-	1    2800 5700
+P 2850 6050
+F 0 "C4" H 2735 6004 50  0000 R CNN
+F 1 "1u" H 2735 6095 50  0000 R CNN
+F 2 "Capacitor_SMD:C_0805_2012Metric_Pad1.15x1.40mm_HandSolder" H 2888 5900 50  0001 C CNN
+F 3 "~" H 2850 6050 50  0001 C CNN
+	1    2850 6050
 	-1   0    0    1
 $EndComp
 Wire Wire Line
-	2350 5500 2350 5550
-Wire Wire Line
-	2350 5400 2800 5400
-Wire Wire Line
-	2800 5400 2800 5300
-Wire Wire Line
-	2800 5400 2800 5550
-Connection ~ 2800 5400
-Connection ~ 1600 5400
-Wire Wire Line
-	2050 5850 2050 5800
+	2400 5850 2400 5900
+Wire Wire Line
+	2400 5750 2850 5750
+Wire Wire Line
+	2850 5750 2850 5650
+Wire Wire Line
+	2850 5750 2850 5900
+Connection ~ 2850 5750
+Connection ~ 1650 5750
+Wire Wire Line
+	2100 6200 2100 6150
 $Comp
 L power:VBUS #PWR04
@@
 Text Notes 9100 6450 0    50   ~ 0
 Typically used diodes:\n- 1N5819: in SOD123F or DO-41\n- LSM115JE3/TR13 : DO-214BA\n- BAS70 : in SOT23\n- 1N4448 : in SOD123\n- BAT54C : in SOT-23 : WeAct F4x1 DevBoards
-Text Notes 700  6500 0    50   ~ 0
-Some clones uses AMS1117 as Linear Voltage Regulator\nwith tantalum SMD capacitors:\n- Pre-capacitor\n- Post-capacitor
+Text Notes 750  6850 0    50   ~ 0
+Some clones uses AMS1117 as Linear Voltage Regulator\nwith tantalum SMD capacitors:\n- Pre-capacitor: 7343 Metric Package : \n- Post-capacitor: 7343 Metric Package :
 Text Notes 9100 5950 0    50   ~ 0
 Not Present on original BluePill.\nHighly recomended.
@@
 Wire Wire Line
 	9150 5050 9150 4950
+Text Notes 550  4200 0    50   ~ 0
+Another suggestion is to use polymer resettable fuse like:\n- case 1210 (inch) : from Samsung Tab batteries\n- case 1206 : typically used on ST-Link clones
 $EndSCHEMATC

Commit message: Updates
Other:
- moved on the sheet: C1, C10, C11, C12, C13, C14, C15, C2, C3, C4, C5, C6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

Commit message: minor updates
Parts:
- added F1: 500mA, Fuse:Fuse_1206_3216Metric, symbol Device:Polyfuse
- C1, C4: footprint Capacitor_SMD:C_0805_2012Metric_Pad1.15x1.40mm_HandSolder -> Capacitor_SMD:C_0805_2012Metric
- C10: renamed from C15; footprint Capacitor_SMD:C_0603_1608Metric_Pad1.05x0.95mm_HandSolder -> Capacitor_SMD:C_0603_1608Metric
- C11, C12, C2, C3, C5, C6, C7: footprint Capacitor_SMD:C_0603_1608Metric_Pad1.05x0.95mm_HandSolder -> Capacitor_SMD:C_0603_1608Metric
- C13: renamed from C10; footprint Capacitor_SMD:C_0603_1608Metric_Pad1.05x0.95mm_HandSolder -> Capacitor_SMD:C_0603_1608Metric
- C14: renamed from C13; footprint Capacitor_SMD:C_0603_1608Metric_Pad1.05x0.95mm_HandSolder -> Capacitor_SMD:C_0603_1608Metric
- C15: renamed from C14; footprint Capacitor_SMD:C_0603_1608Metric_Pad1.05x0.95mm_HandSolder -> Capacitor_SMD:C_0603_1608Metric
- C8: renamed from C9; footprint Capacitor_SMD:C_0603_1608Metric_Pad1.05x0.95mm_HandSolder -> Capacitor_SMD:C_0603_1608Metric
- C9: renamed from C8; footprint Capacitor_SMD:C_0603_1608Metric_Pad1.05x0.95mm_HandSolder -> Capacitor_SMD:C_0603_1608Metric
- D2: renamed from D1; footprint LED_SMD:LED_0603_1608Metric_Pad1.05x0.95mm_HandSolder -> LED_SMD:LED_0603_1608Metric_Castellated
- D3: renamed from D2; footprint LED_SMD:LED_0603_1608Metric_Pad1.05x0.95mm_HandSolder -> LED_SMD:LED_0603_1608Metric_Castellated
- R1, R2, R3, R4, R5, R8, R9: footprint Resistor_SMD:R_0603_1608Metric_Pad1.05x0.95mm_HandSolder -> Resistor_SMD:R_0603_1608Metric
- R6: renamed from R7; footprint Resistor_SMD:R_0603_1608Metric_Pad1.05x0.95mm_HandSolder -> Resistor_SMD:R_0603_1608Metric
- R7: renamed from R6; footprint Resistor_SMD:R_0603_1608Metric_Pad1.05x0.95mm_HandSolder -> Resistor_SMD:R_0603_1608Metric
- U1: footprint Package_TO_SOT_SMD:SOT-353_SC-70-5_Handsoldering -> Package_TO_SOT_SMD:SOT-353_SC-70-5
- renumbered D3 to D1, J5 to J4, J4 to J5
Connections:
- net +3V3: now also J5.18 (Pin_18); no longer J5.3 (Pin_3)
- net +BATT: now also J5.1 (Pin_1); no longer J5.20 (Pin_20)
- net GNDREF: now also J5.19 (Pin_19), J5.20 (Pin_20); no longer J5.1 (Pin_1), J5.2 (Pin_2)
- net NRST: now also J5.17 (Pin_17); no longer J5.4 (Pin_4)
- net PA0: now also J5.5 (Pin_5); no longer J5.16 (Pin_16)
- net PA1: now also J5.6 (Pin_6); no longer J5.15 (Pin_15)
- net PA2: now also J5.7 (Pin_7); no longer J5.14 (Pin_14)
- net PA3: now also J5.8 (Pin_8); no longer J5.13 (Pin_13)
- net PA4: now also J5.9 (Pin_9); no longer J5.12 (Pin_12)
- net PA5: now also J5.10 (Pin_10); no longer J5.11 (Pin_11)
- net PA6: now also J5.11 (Pin_11); no longer J5.10 (Pin_10)
- net PA7: now also J5.12 (Pin_12); no longer J5.9 (Pin_9)
- net PB0: now also J5.13 (Pin_13); no longer J5.8 (Pin_8)
- net PB1: now also J5.14 (Pin_14); no longer J5.7 (Pin_7)
- net PB10: now also J5.15 (Pin_15); no longer J5.6 (Pin_6)
- net PB11: now also J5.16 (Pin_16); no longer J5.5 (Pin_5)
- net PC13: now also J5.2 (Pin_2); no longer J5.19 (Pin_19)
- net PC14: now also J5.3 (Pin_3); no longer J5.18 (Pin_18)
- net PC15: now also J5.4 (Pin_4); no longer J5.17 (Pin_17)
- net VBUS: now also F1.2; no longer C2.1, D1.2 (A)
- new net: C2.1, D1.2 (A), F1.1
Other:
- moved on the sheet: J3, J5
