File: project files/classic/bluepill.kicad_pcb (KiCad board)
At the start: 2 copper layers, 22.9 x 53.3 mm, 35 parts, among them J1 USB_B_Micro, J2 Boot, J3 Left Row, J4 Right Row, J5 SWD, SW1 Reset, U1 RT8183-33, U2 STM32F103C8Tx, Y1 8MHz, Y2 32768Hz

Commit message: re-routing
Parts:
- added C15: 100n, Capacitor_SMD:C_0603_1608Metric_Pad1.05x0.95mm_HandSolder, F.Cu at (123.0, 59.1)
- added D3: SD103AWS, Diode_SMD:D_SOD-323, B.Cu at (109.9, 125.7)
- added D4: BAT54C, Package_TO_SOT_SMD:SOT-23, B.Cu at (156.5, 121.9)
- C5, C6, C7, C8, C9, R1, R5, R8, R9: moved to B.Cu
- D2: value PWR -> Power
- moved J3 83.7 mm to (157.5, 133.3), turned to 90 degrees
- moved C2 76.4 mm to (108.0, 125.7), turned to 270 degrees
- moved C1 76.1 mm to (116.2, 129.3), turned to 90 degrees
- moved J1 74.7 mm to (110.5, 125.7), turned to 270 degrees
- moved C4 74.4 mm to (123.6, 130.2), turned to 180 degrees
- moved D1 74.3 mm to (151.8, 128.3), turned to 270 degrees
- moved SW1 74.1 mm to (119.4, 128.9), turned to 0 degrees
- moved U1 74.1 mm to (119.4, 128.9), turned to 0 degrees
- moved C3 71.7 mm to (123.8, 128.3), turned to 180 degrees
- moved Y2 69.1 mm to (148.0, 125.7), turned to 90 degrees
- moved J2 68.5 mm to (121.9, 121.3), turned to 270 degrees
- moved R6 67.3 mm to (142.2, 125.7), turned to 90 degrees
- moved D2 67.1 mm to (151.8, 123.0), turned to 270 degrees
- moved J5 66.7 mm to (153.7, 121.9), turned to 0 degrees
- moved U2 66.5 mm to (133.3, 125.7), turned to 225 degrees
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Connections:
- C2 pad 1: +5V -> VBUS
- C6 pad 1: PC14 -> PC15
- C8 pad 1: PC15 -> PC14
- J1 pad 1: +5V -> VBUS
- U2 pad 1: +BATT -> Vbat_protected
- Y2 pad 1: PC14 -> PC15
- Y2 pad 4: PC15 -> PC14
Routing:
- net PC15: track 0.00 -> 17.4 mm, vias 0 -> 1
- net OSCIN: track 0.00 -> 14.1 mm
- net PC14: track 0.00 -> 13.5 mm, vias 0 -> 1
- net OSCOUT: track 0.00 -> 12.4 mm
Other:
- board size 22.9 x 53.3 mm -> 53.3 x 22.9 mm

Commit message: Update bluepill.kicad_pcb
Parts:
- C10, C11, C14, C15, R2, R3, R4: moved to B.Cu
- moved C15 73.6 mm to (156.6, 124.5), turned to 180 degrees
- moved C12 67.6 mm to (119.9, 147.2)
- moved C13 67.6 mm to (124.3, 147.2)
- moved C10 57.9 mm to (156.5, 129.5), turned to 180 degrees
- moved C11 54.8 mm to (134.6, 129.5), turned to 270 degrees
- moved R3 53.3 mm to (132.7, 126.1), turned to 90 degrees
- moved C14 46.2 mm to (134.6, 122.6), turned to 270 degrees
- moved R7 38.6 mm to (125.3, 126.4), turned to 180 degrees
- moved R2 38.2 mm to (130.8, 126.1), turned to 270 degrees
- moved R4 36.1 mm to (134.6, 126.1), turned to 90 degrees
- moved C4 0.89 mm to (124.5, 130.0)
- moved C1 0.64 mm to (115.6, 129.3)
- moved C9 0.64 mm to (127.0, 129.5)
- moved C2 0.63 mm to (108.6, 125.7)
- moved C3 0.63 mm to (124.5, 128.3)
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Routing:
- net PC15: track 17.4 -> 0.00 mm, vias 1 -> 0
- net OSCIN: track 14.1 -> 0.00 mm
- net PC14: track 13.5 -> 0.00 mm, vias 1 -> 0
- net OSCOUT: track 12.4 -> 0.00 mm
Other:
- board text added: "3.3"
- board text added: "A0"
- board text added: "A1"
- board text added: "A10"
- board text added: "A11"
- board text added: "A12"
- board text added: "A15"
- board text added: "A2"
- board text added: "A3"
- board text added: "A4"
- board text added: "A5"
- board text added: "A6"
- board text added: "A7"
- board text added: "A8"
- board text added: "A9"
- board text added: "B0"
- board text added: "B1"
- board text added: "B10"
- board text added: "B11"
- board text added: "B12"
- board text added: "B13"
- board text added: "B14"
- board text added: "B15"
- board text added: "B3"
- board text added: "B4"
- board text added: "B5"
- board text added: "B6"
- board text added: "B7"
- board text added: "B8"
- board text added: "B9"
- board text added: "C13"
- board text added: "C14"
- board text added: "C15"
- board text added: "CLK"
- board text added: "DIO"
- board text added: "G"
- board text added: "GND"
- board text added: "R"
- board text added: "VB"
- board text added: "Vin"

Commit message: Updates
Parts:
- C12, C13: moved to B.Cu
- moved C13 27.6 mm to (136.5, 122.6), turned to 270 degrees
- moved C12 21.8 mm to (132.7, 129.5), turned to 270 degrees
- moved C3 1.27 mm to (123.2, 128.3)
- moved C4 1.27 mm to (123.2, 130.0)
- moved R5 0.64 mm to (125.5, 123.2)
- moved R7 0.64 mm to (125.3, 127.0), turned to 0 degrees
- moved C1 0.63 mm to (114.9, 129.3)
- moved R1 0.63 mm to (125.5, 120.7)
- moved U1 0.63 mm to (118.7, 128.9)
- moved Y1 0.13 mm to (142.1, 123.2)
- moved Y2 0.13 mm to (147.8, 125.7)

Commit message: minor
Parts:
- moved C12 1.80 mm to (131.4, 128.3)
- moved C11 1.03 mm to (134.6, 128.5)
Routing:
- net PA0: track 0.00 -> 13.7 mm
- net PB11: track 0.00 -> 12.2 mm
- net PA1: track 0.00 -> 11.4 mm
- net PB10: track 0.00 -> 9.91 mm
- net PA2: track 0.00 -> 9.15 mm
- net PA3: track 0.00 -> 8.48 mm
- net PB1: track 0.00 -> 8.28 mm
- net PA4: track 0.00 -> 8.02 mm
- net PA5: track 0.00 -> 6.27 mm
- net PB0: track 0.00 -> 5.98 mm
- net PA6: track 0.00 -> 4.81 mm
- net PA7: track 0.00 -> 4.72 mm
Other:
- net class Default: trace_width 0.25 -> 0.2; via_dia 0.8 -> 0.5; via_drill 0.4 -> 0.3
Changed lines of the file:
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@@
     (thickness 1.6)
     (drawings 48)
-    (tracks 0)
+    (tracks 70)
     (zones 0)
     (modules 38)
@@
   )
   (setup
-    (last_trace_width 0.25)
+    (last_trace_width 0.2)
     (trace_clearance 0.2)
     (zone_clearance 0.508)
     (zone_45_only no)
     (trace_min 0.2)
-    (via_size 0.8)
-    (via_drill 0.4)
+    (via_size 0.5)
+    (via_drill 0.3)
     (via_min_size 0.4)
     (via_min_drill 0.3)
@@
     (edge_width 0.05)
     (segment_width 0.2)
-    (pcb_text_width 0.3)
-    (pcb_text_size 1.5 1.5)
+    (pcb_text_width 0.25)
+    (pcb_text_size 1.3 1.3)
     (mod_edge_width 0.12)
-    (mod_text_size 1 1)
-    (mod_text_width 0.15)
+    (mod_text_size 1.3 1.3)
+    (mod_text_width 0.25)
     (pad_size 1.524 1.524)
     (pad_drill 0.762)
@@
   (net_class Default "This is the default net class."
     (clearance 0.2)
-    (trace_width 0.25)
-    (via_dia 0.8)
-    (via_drill 0.4)
+    (trace_width 0.2)
+    (via_dia 0.5)
+    (via_drill 0.3)
     (uvia_dia 0.3)
     (uvia_drill 0.1)
@@
   )
   (module Capacitor_SMD:C_0603_1608Metric_Pad1.05x0.95mm_HandSolder (layer B.Cu)
-    (at 132.715 129.54 270)
+    (at 131.445 128.27 270)
     (descr "Capacitor SMD 0603 (1608 Metric), square (rectangular) end terminal, IPC_7351 nominal with elongated pad for handsoldering. (Body size source: http://www.tortai-tech.com/upload/download/2011102023233369053.pdf), generated with kicad-footprint-generator")
     (tags "capacitor handsolder")
@@
   )
   (module Capacitor_SMD:C_0603_1608Metric_Pad1.05x0.95mm_HandSolder (layer B.Cu)
-    (at 134.62 129.54 270)
+    (at 134.62 128.51 270)
     (descr "Capacitor SMD 0603 (1608 Metric), square (rectangular) end terminal, IPC_7351 nominal with elongated pad for handsoldering. (Body size source: http://www.tortai-tech.com/upload/download/2011102023233369053.pdf), generated with kicad-footprint-generator")
     (tags "capacitor handsolder")
@@
   )
   (gr_text A4 (at 137.16 115.57) (layer F.SilkS)
-    (effects (font (size 0.889 0.889) (thickness 0.1524)))
+    (effects (font (size 1.25 1.25) (thickness 0.25)))
   )
   (gr_text A5 (at 134.62 115.57) (layer F.SilkS)
@@
   (gr_line (start 106.68 114.3) (end 160.02 114.3) (layer Edge.Cuts) (width 0.05))
   (gr_line (start 106.68 137.16) (end 106.68 114.3) (layer Edge.Cuts) (width 0.05))
+  (segment (start 135.701126 120.904) (end 135.055895 121.549231) (width 0.2) (layer F.Cu) (net 35))
+  (segment (start 137.229986 120.904) (end 135.701126 120.904) (width 0.2) (layer F.Cu) (net 35))
+  (segment (start 138.924988 120.49201) (end 137.641976 120.49201) (width 0.2) (layer F.Cu) (net 35))
+  (segment (start 139.274998 120.142) (end 138.924988 120.49201) (width 0.2) (layer F.Cu) (net 35))
+  (segment (start 141.32001 120.142) (end 139.274998 120.142) (width 0.2) (layer F.Cu) (net 35))
+  (segment (start 146.05 119.38) (end 144.004988 119.38) (width 0.2) (layer F.Cu) (net 35))
+  (segment (start 147.32 118.11) (end 146.05 119.38) (width 0.2) (layer F.Cu) (net 35))
+  (segment (start 137.641976 120.49201) (end 137.229986 120.904) (width 0.2) (layer F.Cu) (net 35))
+  (segment (start 144.004988 119.38) (end 143.654978 119.73001) (width 0.2) (layer F.Cu) (net 35))
+  (segment (start 143.654978 119.73001) (end 141.732 119.73001) (width 0.2) (layer F.Cu) (net 35))
+  (segment (start 141.732 119.73001) (end 141.32001 120.142) (width 0.2) (layer F.Cu) (net 35))
+  (segment (start 135.40601 120.49201) (end 134.702342 121.195678) (width 0.2) (layer F.Cu) (net 36))
+  (segment (start 137.146988 120.49201) (end 135.40601 120.49201) (width 0.2) (layer F.Cu) (net 36))
+  (segment (start 137.496998 120.142) (end 137.146988 120.49201) (width 0.2) (layer F.Cu) (net 36))
+  (segment (start 141.464988 119.38) (end 141.114978 119.73001) (width 0.2) (layer F.Cu) (net 36))
+  (segment (start 138.78001 120.142) (end 137.496998 120.142) (width 0.2) (layer F.Cu) (net 36))
+  (segment (start 143.51 119.38) (end 141.464988 119.38) (width 0.2) (layer F.Cu) (net 36))
+  (segment (start 144.78 118.11) (end 143.51 119.38) (width 0.2) (layer F.Cu) (net 36))
+  (segment (start 141.114978 119.73001) (end 139.192 119.73001) (width 0.2) (layer F.Cu) (net 36))
+  (segment (start 139.192 119.73001) (end 138.78001 120.142) (width 0.2) (layer F.Cu) (net 36))
+  (segment (start 134.83678 120.142) (end 134.348788 120.629992) (width 0.2) (layer F.Cu) (net 37))
+  (segment (start 137.00201 120.142) (end 134.83678 120.142) (width 0.2) (layer F.Cu) (net 37))
+  (segment (start 142.24 118.11) (end 140.97 119.38) (width 0.2) (layer F.Cu) (net 37))
+  (segment (start 134.348788 120.629992) (end 134.348788 120.842124) (width 0.2) (layer F.Cu) (net 37))
+  (segment (start 140.97 119.38) (end 138.924988 119.38) (width 0.2) (layer F.Cu) (net 37))
+  (segment (start 138.924988 119.38) (end 138.574978 119.73001) (width 0.2) (layer F.Cu) (net 37))
+  (segment (start 138.574978 119.73001) (end 137.414 119.73001) (width 0.2) (layer F.Cu) (net 37))
+  (segment (start 137.414 119.73001) (end 137.00201 120.142) (width 0.2) (layer F.Cu) (net 37))
+  (segment (start 134.62 119.73001) (end 136.80999 119.73001) (width 0.2) (layer F.Cu) (net 38))
+  (segment (start 136.80999 119.73001) (end 137.16 119.38) (width 0.2) (layer F.Cu) (net 38))
+  (segment (start 139.7 118.11) (end 138.43 119.38) (width 0.2) (layer F.Cu) (net 38))
+  (segment (start 138.43 119.38) (end 137.16 119.38) (width 0.2) (layer F.Cu) (net 38))
+  (segment (start 134.62 119.73001) (end 134.20801 120.142) (width 0.2) (layer F.Cu) (net 38))
+  (segment (start 133.051336 120.142) (end 132.351212 120.842124) (width 0.2) (layer F.Cu) (net 38))
+  (segment (start 134.20801 120.142) (end 133.051336 120.142) (width 0.2) (layer F.Cu) (net 38))
+  (segment (start 136.310001 118.959999) (end 137.16 118.11) (width 0.2) (layer F.Cu) (net 39))
+  (segment (start 134.366 119.38) (end 135.89 119.38) (width 0.2) (layer F.Cu) (net 39))
+  (segment (start 131.318 120.51602) (end 131.318 120.142) (width 0.2) (layer F.Cu) (net 39))
+  (segment (start 135.89 119.38) (end 136.310001 118.959999) (width 0.2) (layer F.Cu) (net 39))
+  (segment (start 131.997658 121.195678) (end 131.318 120.51602) (width 0.2) (layer F.Cu) (net 39))
+  (segment (start 134.01599 119.73001) (end 134.366 119.38) (width 0.2) (layer F.Cu) (net 39))
+  (segment (start 131.318 120.142) (end 131.72999 119.73001) (width 0.2) (layer F.Cu) (net 39))
+  (segment (start 131.72999 119.73001) (end 134.01599 119.73001) (width 0.2) (layer F.Cu) (net 39))
+  (segment (start 133.35 119.38) (end 134.62 118.11) (width 0.2) (layer F.Cu) (net 40))
+  (segment (start 130.96799 119.997022) (end 131.585012 119.38) (width 0.2) (layer F.Cu) (net 40))
+  (segment (start 131.585012 119.38) (end 133.35 119.38) (width 0.2) (layer F.Cu) (net 40))
+  (segment (start 131.644105 121.549231) (end 130.96799 120.873116) (width 0.2) (layer F.Cu) (net 40))
+  (segment (start 130.96799 120.873116) (end 130.96799 119.997022) (width 0.2) (layer F.Cu) (net 40))
+  (segment (start 131.149145 121.902785) (end 130.556 121.30964) (width 0.2) (layer F.Cu) (net 41))
+  (segment (start 131.290551 121.902785) (end 131.149145 121.902785) (width 0.2) (layer F.Cu) (net 41))
+  (segment (start 130.556 119.634) (end 132.08 118.11) (width 0.2) (layer F.Cu) (net 41))
+  (segment (start 130.556 121.30964) (end 130.556 119.634) (width 0.2) (layer F.Cu) (net 41))
+  (segment (start 129.54 120.85934) (end 130.936998 122.256338) (width 0.2) (layer F.Cu) (net 42))
+  (segment (start 129.54 118.11) (end 129.54 120.85934) (width 0.2) (layer F.Cu) (net 42))
+  (segment (start 130.583445 122.609891) (end 129.032 121.058446) (width 0.2) (layer F.Cu) (net 43))
+  (segment (start 129.032 120.142) (end 127 118.11) (width 0.2) (layer F.Cu) (net 43))
+  (segment (start 129.032 121.058446) (end 129.032 120.142) (width 0.2) (layer F.Cu) (net 43))
+  (segment (start 128.609501 121.343055) (end 130.229891 122.963445) (width 0.2) (layer F.Cu) (net 44))
+  (segment (start 128.609501 120.481501) (end 128.609501 121.343055) (width 0.2) (layer F.Cu) (net 44))
+  (segment (start 127.508 119.38) (end 128.609501 120.481501) (width 0.2) (layer F.Cu) (net 44))
+  (segment (start 125.73 119.38) (end 127.508 119.38) (width 0.2) (layer F.Cu) (net 44))
+  (segment (start 124.46 118.11) (end 125.73 119.38) (width 0.2) (layer F.Cu) (net 44))
+  (segment (start 125.232234 119.38) (end 129.522785 123.670551) (width 0.2) (layer F.Cu) (net 45))
+  (segment (start 121.92 118.11) (end 123.19 119.38) (width 0.2) (layer F.Cu) (net 45))
+  (segment (start 123.19 119.38) (end 125.232234 119.38) (width 0.2) (layer F.Cu) (net 45))
+  (segment (start 123.045022 119.73001) (end 124.875136 119.73001) (width 0.2) (layer F.Cu) (net 46))
+  (segment (start 122.695012 119.38) (end 123.045022 119.73001) (width 0.2) (layer F.Cu) (net 46))
+  (segment (start 119.38 118.11) (end 120.65 119.38) (width 0.2) (layer F.Cu) (net 46))
+  (segment (start 124.875136 119.73001) (end 129.169231 124.024105) (width 0.2) (layer F.Cu) (net 46))
+  (segment (start 120.65 119.38) (end 122.695012 119.38) (width 0.2) (layer F.Cu) (net 46))
 )

Commit message: minor updates
Parts:
- added F1: 500mA, Fuse:Fuse_1206_3216Metric, B.Cu at (109.2, 125.0)
- C1, C4: footprint Capacitor_SMD:C_0805_2012Metric_Pad1.15x1.40mm_HandSolder -> Capacitor_SMD:C_0805_2012Metric
- C10, C11, C12, C13, C14, C15, C2, C3, C5, C6, C7: footprint Capacitor_SMD:C_0603_1608Metric_Pad1.05x0.95mm_HandSolder -> Capacitor_SMD:C_0603_1608Metric
- C8: value 20pF -> 100nF; footprint Capacitor_SMD:C_0603_1608Metric_Pad1.05x0.95mm_HandSolder -> Capacitor_SMD:C_0603_1608Metric
- C9: value 100nF -> 20pF; footprint Capacitor_SMD:C_0603_1608Metric_Pad1.05x0.95mm_HandSolder -> Capacitor_SMD:C_0603_1608Metric
- D1: value PC13 -> SD103AWS; footprint LED_SMD:LED_0603_1608Metric_Pad1.05x0.95mm_HandSolder -> Diode_SMD:D_SOD-323
- D2: value Power -> PC13; footprint LED_SMD:LED_0603_1608Metric_Pad1.05x0.95mm_HandSolder -> LED_SMD:LED_0603_1608Metric_Castellated
- D3: value SD103AWS -> Power; footprint Diode_SMD:D_SOD-323 -> LED_SMD:LED_0603_1608Metric_Castellated
- J4: value Right Row -> SWD; footprint Connector_PinHeader_2.54mm:PinHeader_1x20_P2.54mm_Vertical -> Connector_PinHeader_2.54mm:PinHeader_1x04_P2.54mm_Horizontal; moved to F.Cu
- J5: value SWD -> Right Row; footprint Connector_PinHeader_2.54mm:PinHeader_1x04_P2.54mm_Horizontal -> Connector_PinHeader_2.54mm:PinHeader_1x20_P2.54mm_Vertical; moved to B.Cu
- R1, R2, R3, R4, R5, R8, R9: footprint Resistor_SMD:R_0603_1608Metric_Pad1.05x0.95mm_HandSolder -> Resistor_SMD:R_0603_1608Metric
- R6: value 10M [N/A] -> 10K; footprint Resistor_SMD:R_0603_1608Metric_Pad1.05x0.95mm_HandSolder -> Resistor_SMD:R_0603_1608Metric
- R7: value 10K -> 10M [N/A]; footprint Resistor_SMD:R_0603_1608Metric_Pad1.05x0.95mm_HandSolder -> Resistor_SMD:R_0603_1608Metric
- U1: footprint Package_TO_SOT_SMD:SOT-353_SC-70-5_Handsoldering -> Package_TO_SOT_SMD:SOT-353_SC-70-5
- moved J4 44.6 mm to (153.7, 121.9), turned to 0 degrees
- moved J5 5.39 mm to (157.5, 118.1), turned to 90 degrees
- moved D3 5.08 mm to (110.7, 130.8), turned to 180 degrees
- moved C2 2.54 mm to (108.7, 128.3), turned to 180 degrees
Connections:
- C10 pad 1: GNDREF -> Vbat_protected
- C10 pad 2: +3V3 -> GNDREF
- C13 pad 1: +3V3 -> GNDREF
- C13 pad 2: GNDREF -> +3V3
- C15 pad 1: Vbat_protected -> +3V3
- C2 pad 1: VBUS -> Net-(C2-Pad1)
- C8 pad 1: PC14 -> NRST
- C9 pad 1: NRST -> PC14
- D1 pad 1: Net-(D1-Pad1) -> +5V
- D1 pad 2: +3V3 -> Net-(C2-Pad1)
- D3 pad 1: +5V -> Net-(D3-Pad1)
- D3 pad 2: VBUS -> +3V3
- J4 pad 2: GNDREF -> SWCLK
- J4 pad 3: +3V3 -> SWDIO
- J4 pad 4: NRST -> +3V3
- J5 pad 1: GNDREF -> +BATT
- J5 pad 2: SWCLK -> PC13
- J5 pad 3: SWDIO -> PC14
- J5 pad 4: +3V3 -> PC15
- R6 pad 1: OSCIN -> NRST
- R6 pad 2: OSCOUT -> +3V3
- R7 pad 1: NRST -> OSCIN
- R7 pad 2: +3V3 -> OSCOUT
- R8 pad 2: Net-(D1-Pad1) -> Net-(D2-Pad1)
- R9 pad 2: Net-(D2-Pad1) -> Net-(D3-Pad1)
Routing:
- net PA0: track 13.7 -> 0.00 mm
- net PB11: track 12.2 -> 0.00 mm
- net PA1: track 11.4 -> 0.00 mm
- net PB10: track 9.91 -> 0.00 mm
- net PA2: track 9.15 -> 0.00 mm
- net PA3: track 8.48 -> 0.00 mm
- net PB1: track 8.28 -> 0.00 mm
- net PA4: track 8.02 -> 0.00 mm
- net PA5: track 6.27 -> 0.00 mm
- net PB0: track 5.98 -> 0.00 mm
- net PA6: track 4.81 -> 0.00 mm
- net PA7: track 4.72 -> 0.00 mm

Commit message: Update bluepill.kicad_pcb
Parts:
- D1, R7: moved to B.Cu
- D3: moved to F.Cu
- moved D3 41.8 mm to (151.8, 123.2), turned to 90 degrees
- moved D1 36.8 mm to (114.9, 128.9), turned to 90 degrees
- moved C8 21.1 mm to (126.4, 127.0), turned to 270 degrees
- moved C9 19.1 mm to (146.1, 130.2), turned to 180 degrees
- moved R6 17.8 mm to (124.5, 127.0), turned to 270 degrees
- moved R7 17.0 mm to (142.2, 125.7), turned to 90 degrees
- moved C14 6.38 mm to (128.3, 121.9)
- moved C6 5.36 mm to (149.2, 130.2), turned to 0 degrees
- moved D2 5.32 mm to (151.8, 128.3)
- moved C15 5.09 mm to (156.4, 129.5), turned to 0 degrees
- moved C10 5.08 mm to (156.4, 124.5), turned to 0 degrees
- moved C2 2.66 mm to (108.0, 125.7), turned to 90 degrees
- moved C12 2.29 mm to (132.7, 130.2)
- moved C1 1.94 mm to (116.8, 128.9), turned to 270 degrees
- moved C3 1.91 mm to (121.9, 126.8), turned to 270 degrees
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Routing:
- added copper zone on B.Cu, net GNDREF
- added copper zone on F.Cu, net GNDREF
Other:
- board text added: "0"
- board text added: "1"
- board text added: "Boot0"

Commit message: Update bluepill.kicad_pcb
Parts:
- moved J2 0.64 mm to (121.9, 121.9)
- moved SW1 0.63 mm to (119.4, 128.9)
Changed lines of the file:
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@@
   )
   (module Button_Switch_SMD:SW_SPST_TL3342 (layer F.Cu)
-    (at 119.38 128.27 180)
+    (at 119.38 128.905 180)
     (descr "Low-profile SMD Tactile Switch, https://www.e-switch.com/system/asset/product_line/data_sheet/165/TL3342.pdf")
     (tags "SPST Tactile Switch")
@@
   )
   (module Connector_PinHeader_2.54mm:PinHeader_2x03_P2.54mm_Vertical (layer F.Cu)
-    (at 121.92 121.285 270)
+    (at 121.92 121.92 270)
     (descr "Through hole straight pin header, 2x03, 2.54mm pitch, double rows")
     (tags "Through hole pin header THT 2x03 2.54mm double row")
@@
   )
   (gr_text Boot0 (at 119.38 120.015) (layer F.SilkS)
-    (effects (font (size 1.3 1.3) (thickness 0.25)))
-  )
-  (gr_text 1 (at 123.825 123.825) (layer F.SilkS)
-    (effects (font (size 1.3 1.3) (thickness 0.25)))
-  )
-  (gr_text 1 (at 123.825 121.285) (layer F.SilkS)
-    (effects (font (size 1.3 1.3) (thickness 0.25)))
-  )
-  (gr_text 0 (at 114.935 123.825) (layer F.SilkS)
-    (effects (font (size 1.3 1.3) (thickness 0.25)))
-  )
-  (gr_text 0 (at 114.935 121.285) (layer F.SilkS)
-    (effects (font (size 1.3 1.3) (thickness 0.25)))
-  )
-  (gr_poly (pts (xy 121.92 132.08) (xy 121.285 130.81) (xy 122.555 130.81)) (layer F.SilkS) (width 0.1))
-  (gr_poly (pts (xy 125.095 132.08) (xy 123.825 132.08) (xy 124.46 130.81)) (layer F.SilkS) (width 0.1))
+    (effects (font (size 1.016 1.016) (thickness 0.1778)))
+  )
+  (gr_text 1 (at 123.825 124.46) (layer F.SilkS)
+    (effects (font (size 1.3 1.3) (thickness 0.25)))
+  )
+  (gr_text 1 (at 123.825 121.92) (layer F.SilkS)
+    (effects (font (size 1.3 1.3) (thickness 0.25)))
+  )
+  (gr_text 0 (at 114.935 124.46) (layer F.SilkS)
+    (effects (font (size 1.3 1.3) (thickness 0.25)))
+  )
+  (gr_text 0 (at 114.935 121.92) (layer F.SilkS)
+    (effects (font (size 1.3 1.3) (thickness 0.25)))
+  )
+  (gr_poly (pts (xy 121.92 132.334) (xy 121.285 131.064) (xy 122.555 131.064)) (layer F.SilkS) (width 0))
+  (gr_poly (pts (xy 125.095 132.334) (xy 123.825 132.334) (xy 124.46 131.064)) (layer F.SilkS) (width 0))
   (gr_text GND (at 159.385 121.92 90) (layer F.SilkS)
     (effects (font (size 0.889 0.889) (thickness 0.1524)))
