File: project files/reforged/bluepill_reforged.sch (KiCad schematic (older format))
At the start: 39 parts, among them J1 USB_C_Receptacle_USB2.0, J2 Left Castellation, J3 Cortex debug, J4 Right Castellation, SW1 Boot0, SW2 Reset, U1 AMS1117-3.3, U2 STM32F103C8Tx, Y1 8MHz, Y2 32768Hz

Commit message: replaced SWD 10 with 14
Parts:
- removed D4, D5: 1N5819, Diode_THT:D_DO-41_SOD81_P10.16mm_Horizontal, symbol Diode:1N5819
- removed J3: Cortex debug, Connector_PinHeader_1.27mm:PinHeader_2x05_P1.27mm_Vertical_SMD, symbol Connector:Conn_ARM_JTAG_SWD_10
- added D4: BAT54C, Package_TO_SOT_SMD:SOT-23, symbol Diode:BAT54C
- added J3: STDC14, Connector_PinHeader_1.27mm:PinHeader_2x07_P1.27mm_Vertical_SMD, symbol Connector_Generic:Conn_02x07_Odd_Even
- C3, C8: value 1uF -> 100nf
- D1: footprint Diode_SMD:D_SMA_Handsoldering -> Diode_SMD:D_SOD-128
- D2: value Green -> PC13
Connections:
- net labels added: RX, TX
- wire segments 120 -> 129
- no-connect marks 5 -> 8
Other:
- note added: "STDC14 interface"
- note removed: "SWD interface"
- moved on the sheet: C9
Changed lines of the file:
@@
 F 0 "D1" H 2000 834 50  0000 C CNN
 F 1 "Protection" H 2000 925 50  0000 C CNN
-F 2 "Diode_SMD:D_SMA_Handsoldering" H 2000 1050 50  0001 C CNN
+F 2 "Diode_SMD:D_SOD-128" H 2000 1050 50  0001 C CNN
 F 3 "~" H 2000 1050 50  0001 C CNN
 	1    2000 1050
@@
 P 3600 2550
 F 0 "C3" H 3715 2596 50  0000 L CNN
-F 1 "1uF" H 3715 2505 50  0000 L CNN
+F 1 "100nf" H 3715 2505 50  0000 L CNN
 F 2 "Capacitor_SMD:C_0603_1608Metric_Pad1.05x0.95mm_HandSolder" H 3638 2400 50  0001 C CNN
 F 3 "~" H 3600 2550 50  0001 C CNN
@@
 P 5900 1150
 F 0 "D2" H 5893 895 50  0000 C CNN
-F 1 "Green" H 5893 986 50  0000 C CNN
+F 1 "PC13" H 5893 986 50  0000 C CNN
 F 2 "LED_SMD:LED_0805_2012Metric_Castellated" H 5900 1150 50  0001 C CNN
 F 3 "~" H 5900 1150 50  0001 C CNN
@@
 Wire Wire Line
 	9450 6250 9450 6350
-Text GLabel 9500 2450 0    50   Input ~ 0
+Text GLabel 9250 2600 0    50   Input ~ 0
 SWO
-Text GLabel 9650 2450 2    50   Input ~ 0
+Text GLabel 9400 2600 2    50   Input ~ 0
 PB3
 Text Notes 9600 2150 0    100  Italic 20
-SWD interface
+STDC14 interface
 $Comp
 L power:+BATT #PWR040
@@
 L power:+BATT #PWR025
 U 1 1 5E61C7BB
-P 7200 5250
-F 0 "#PWR025" H 7200 5100 50  0001 C CNN
-F 1 "+BATT" H 7215 5423 50  0000 C CNN
-F 2 "" H 7200 5250 50  0001 C CNN
-F 3 "" H 7200 5250 50  0001 C CNN
-	1    7200 5250
+P 7550 5350
+F 0 "#PWR025" H 7550 5200 50  0001 C CNN
+F 1 "+BATT" H 7565 5523 50  0000 C CNN
+F 2 "" H 7550 5350 50  0001 C CNN
+F 3 "" H 7550 5350 50  0001 C CNN
+	1    7550 5350
 	1    0    0    -1
 $EndComp
@@
 L power:+3.3V #PWR026
 U 1 1 5E61D33E
-P 7650 5250
-F 0 "#PWR026" H 7650 5100 50  0001 C CNN
-F 1 "+3.3V" H 7665 5378 50  0000 L CNN
-F 2 "" H 7650 5250 50  0001 C CNN
-F 3 "" H 7650 5250 50  0001 C CNN
-	1    7650 5250
-	1    0    0    -1
-$EndComp
-$Comp
-L Diode:1N5819 D5
-U 1 1 5E61DE4A
-P 7650 5400
-F 0 "D5" V 7696 5321 50  0000 R CNN
-F 1 "1N5819" V 7605 5321 50  0000 R CNN
-F 2 "Diode_THT:D_DO-41_SOD81_P10.16mm_Horizontal" H 7650 5225 50  0001 C CNN
-F 3 "http://www.vishay.com/docs/88525/1n5817.pdf" H 7650 5400 50  0001 C CNN
-	1    7650 5400
-	0    -1   -1   0
+P 8150 5350
+F 0 "#PWR026" H 8150 5200 50  0001 C CNN
+F 1 "+3.3V" H 8165 5478 50  0000 L CNN
+F 2 "" H 8150 5350 50  0001 C CNN
+F 3 "" H 8150 5350 50  0001 C CNN
+	1    8150 5350
+	1    0    0    -1
 $EndComp
 $Comp
 L Device:C C9
 U 1 1 5E61F79C
-P 7650 5700
-F 0 "C9" H 7765 5746 50  0000 L CNN
-F 1 "100n" H 7765 5655 50  0000 L CNN
-F 2 "Capacitor_SMD:C_0603_1608Metric_Pad1.05x0.95mm_HandSolder" H 7688 5550 50  0001 C CNN
-F 3 "~" H 7650 5700 50  0001 C CNN
-	1    7650 5700
+P 7850 5700
+F 0 "C9" H 7965 5746 50  0000 L CNN
+F 1 "100n" H 7965 5655 50  0000 L CNN
+F 2 "Capacitor_SMD:C_0603_1608Metric_Pad1.05x0.95mm_HandSolder" H 7888 5550 50  0001 C CNN
+F 3 "~" H 7850 5700 50  0001 C CNN
+	1    7850 5700
 	1    0    0    -1
 $EndComp
@@
 L power:GNDREF #PWR027
 U 1 1 5E620338
-P 7650 5850
-F 0 "#PWR027" H 7650 5600 50  0001 C CNN
-F 1 "GNDREF" H 7655 5677 50  0000 C CNN
-F 2 "" H 7650 5850 50  0001 C CNN
-F 3 "" H 7650 5850 50  0001 C CNN
-	1    7650 5850
-	1    0    0    -1
-$EndComp
-Text GLabel 8000 5550 2    50   Input ~ 0
+P 7850 5850
+F 0 "#PWR027" H 7850 5600 50  0001 C CNN
+F 1 "GNDREF" H 7855 5677 50  0000 C CNN
+F 2 "" H 7850 5850 50  0001 C CNN
+F 3 "" H 7850 5850 50  0001 C CNN
+	1    7850 5850
+	1    0    0    -1
+$EndComp
+Text GLabel 8200 5550 2    50   Input ~ 0
 VBAT_Protected
 Text GLabel 7850 900  2    50   Input ~ 0
@@
 	7750 900  7750 1050
 Wire Wire Line
-	7650 5550 8000 5550
-Connection ~ 7650 5550
+	7850 5550 8200 5550
 Text Notes 7250 5000 0    100  Italic 20
 RTC Power Protection
@@
 P 6200 3000
 F 0 "C8" H 6315 3046 50  0000 L CNN
-F 1 "1uF" H 6315 2955 50  0000 L CNN
+F 1 "100nf" H 6315 2955 50  0000 L CNN
 F 2 "Capacitor_SMD:C_0603_1608Metric_Pad1.05x0.95mm_HandSolder" H 6238 2850 50  0001 C CNN
 F 3 "~" H 6200 3000 50  0001 C CNN
@@
 NoConn ~ 4850 1350
 NoConn ~ 4850 950
-$Comp
-L Diode:1N5819 D4
-U 1 1 5E15A95B
-P 7200 5400
-F 0 "D4" V 7246 5321 50  0000 R CNN
-F 1 "1N5819" V 7155 5321 50  0000 R CNN
-F 2 "Diode_THT:D_DO-41_SOD81_P10.16mm_Horizontal" H 7200 5225 50  0001 C CNN
-F 3 "http://www.vishay.com/docs/88525/1n5817.pdf" H 7200 5400 50  0001 C CNN
-	1    7200 5400
-	0    -1   -1   0
-$EndComp
-Wire Wire Line
-	7200 5550 7650 5550
-Text GLabel 9500 2550 0    50   Input ~ 0
+Text GLabel 9250 2700 0    50   Input ~ 0
 SWDIO
-Text GLabel 9500 2650 0    50   Input ~ 0
+Text GLabel 9250 2800 0    50   Input ~ 0
 SWCLK
 Text GLabel 8550 3650 2    50   Input ~ 0
 PA13
-Text GLabel 9650 2550 2    50   Input ~ 0
+Text GLabel 9400 2700 2    50   Input ~ 0
 PA13
-Text GLabel 9650 2650 2    50   Input ~ 0
+Text GLabel 9400 2800 2    50   Input ~ 0
 PA14
-$Comp
-L power:+3.3V #PWR037
-U 1 1 5E177ECC
-P 10350 2350
-F 0 "#PWR037" H 10350 2200 50  0001 C CNN
-F 1 "+3.3V" H 10365 2478 50  0000 L CNN
-F 2 "" H 10350 2350 50  0001 C CNN
-F 3 "" H 10350 2350 50  0001 C CNN
-	1    10350 2350
-	1    0    0    -1
-$EndComp
-NoConn ~ 10850 3150
-Text GLabel 10850 3050 2    50   Input ~ 0
-SWO
-Text GLabel 10850 2950 2    50   Input ~ 0
-SWDIO
-Text GLabel 10850 2850 2    50   Input ~ 0
-SWCLK
-Text GLabel 10850 2650 2    50   Input ~ 0
-NRST
-$Comp
-L Connector:Conn_ARM_JTAG_SWD_10 J3
-U 1 1 5E16EB42
-P 10350 2950
-F 0 "J3" H 9906 2996 50  0000 R CNN
-F 1 "Cortex debug" H 9906 2905 50  0000 R CNN
-F 2 "Connector_PinHeader_1.27mm:PinHeader_2x05_P1.27mm_Vertical_SMD" H 10350 2950 50  0001 C CNN
-F 3 "http://infocenter.arm.com/help/topic/com.arm.doc.ddi0314h/DDI0314H_coresight_components_trm.pdf" V 10000 1700 50  0001 C CNN
-	1    10350 2950
-	1    0    0    -1
-$EndComp
-$Comp
-L power:GNDREF #PWR038
-U 1 1 5E1809F7
-P 10350 3550
-F 0 "#PWR038" H 10350 3300 50  0001 C CNN
-F 1 "GNDREF" H 10355 3377 50  0000 C CNN
-F 2 "" H 10350 3550 50  0001 C CNN
-F 3 "" H 10350 3550 50  0001 C CNN
-	1    10350 3550
-	1    0    0    -1
-$EndComp
-Wire Wire Line
-	10250 3550 10350 3550
-Connection ~ 10350 3550
 Wire Notes Line
 	6750 500  6750 3950
 Wire Wire Line
-	9650 2450 9500 2450
-Wire Wire Line
-	9500 2550 9650 2550
-Wire Wire Line
-	9650 2650 9500 2650
+	9400 2600 9250 2600
+Wire Wire Line
+	9250 2700 9400 2700
+Wire Wire Line
+	9400 2800 9250 2800
+$Comp
+L Diode:BAT54C D4
+U 1 1 5E16540C
+P 7850 5350
+F 0 "D4" H 7850 5575 50  0000 C CNN
+F 1 "BAT54C" H 7850 5484 50  0000 C CNN
+F 2 "Package_TO_SOT_SMD:SOT-23" H 7925 5475 50  0001 L CNN
+F 3 "http://www.diodes.com/_files/datasheets/ds11005.pdf" H 7770 5350 50  0001 C CNN
+	1    7850 5350
+	1    0    0    -1
+$EndComp
+Connection ~ 7850 5550
+$Comp
+L Connector_Generic:Conn_02x07_Odd_Even J3
+U 1 1 5E19328C
+P 10500 2900
+F 0 "J3" H 10550 3417 50  0000 C CNN
+F 1 "STDC14" H 10550 3326 50  0000 C CNN
+F 2 "Connector_PinHeader_1.27mm:PinHeader_2x07_P1.27mm_Vertical_SMD" H 10500 2900 50  0001 C CNN
+F 3 "~" H 10500 2900 50  0001 C CNN
+	1    10500 2900
+	1    0    0    -1
+$EndComp
+NoConn ~ 10300 2600
+NoConn ~ 10800 2600
+Text GLabel 10800 2800 2    50   Input ~ 0
+SWCLK
+Text GLabel 10800 3100 2    50   Input ~ 0
+NRST
+Text GLabel 10800 2700 2    50   Input ~ 0
+SWDIO
+$Comp
+L power:+3.3V #PWR037
+U 1 1 5E1A21E5
+P 9900 2500
+F 0 "#PWR037" H 9900 2350 50  0001 C CNN
+F 1 "+3.3V" H 9915 2628 50  0000 L CNN
+F 2 "" H 9900 2500 50  0001 C CNN
+F 3 "" H 9900 2500 50  0001 C CNN
+	1    9900 2500
+	1    0    0    -1
+$EndComp
+Wire Wire Line
+	10300 2700 9900 2700
+Wire Wire Line
+	9900 2700 9900 2500
+Text GLabel 10800 2900 2    50   Input ~ 0
+SWO
+NoConn ~ 10800 3000
+NoConn ~ 10300 3000
+Wire Wire Line
+	10300 2800 10200 2800
+Wire Wire Line
+	10200 2800 10200 2900
+Wire Wire Line
+	10200 2900 10300 2900
+Wire Wire Line
+	10300 3100 10200 3100
+Wire Wire Line
+	10200 3100 10200 2900
+Connection ~ 10200 2900
+$Comp
+L power:GNDREF #PWR038
+U 1 1 5E1B90CD
+P 9900 2900
+F 0 "#PWR038" H 9900 2650 50  0001 C CNN
+F 1 "GNDREF" H 9905 2727 50  0000 C CNN
+F 2 "" H 9900 2900 50  0001 C CNN
+F 3 "" H 9900 2900 50  0001 C CNN
+	1    9900 2900
+	1    0    0    -1
+$EndComp
+Wire Wire Line
+	10200 2800 9900 2800
+Wire Wire Line
+	9900 2800 9900 2900
+Connection ~ 10200 2800
+Text GLabel 10800 3200 2    50   Output ~ 0
+TX
+Text GLabel 10300 3200 0    50   Input ~ 0
+RX
+Text GLabel 9250 2900 0    50   Input ~ 0
+RX
+Text GLabel 9250 3000 0    50   Output ~ 0
+TX
+Text GLabel 9400 3000 2    50   Input ~ 0
+PA9
+Text GLabel 9400 2900 2    50   Input ~ 0
+PA10
+Wire Wire Line
+	9250 2900 9400 2900
+Wire Wire Line
+	9250 3000 9400 3000
 $EndSCHEMATC

Commit message: minor
Parts:
- added C14: 100n, Capacitor_SMD:C_0603_1608Metric_Pad1.05x0.95mm_HandSolder, symbol Device:C
Connections:
- net +3V3: now also J4.18 (Pin_18); no longer J4.3 (Pin_3)
- net +BATT: now also J4.1 (Pin_1); no longer J4.20 (Pin_20)
- net GNDREF: now also J4.19 (Pin_19), J4.20 (Pin_20), C14.2; no longer J4.1 (Pin_1), J4.2 (Pin_2)
- net NRST: now also J4.17 (Pin_17); no longer J4.4 (Pin_4)
- net PA0: now also J4.5 (Pin_5); no longer J4.16 (Pin_16)
- net PA1: now also J4.6 (Pin_6); no longer J4.15 (Pin_15)
- net PA2: now also J4.7 (Pin_7); no longer J4.14 (Pin_14)
- net PA3: now also J4.8 (Pin_8); no longer J4.13 (Pin_13)
- net PA4: now also J4.9 (Pin_9); no longer J4.12 (Pin_12)
- net PA5: now also J4.10 (Pin_10); no longer J4.11 (Pin_11)
- net PA6: now also J4.11 (Pin_11); no longer J4.10 (Pin_10)
- net PA7: now also J4.12 (Pin_12); no longer J4.9 (Pin_9)
- net PB0: now also J4.13 (Pin_13); no longer J4.8 (Pin_8)
- net PB1: now also J4.14 (Pin_14); no longer J4.7 (Pin_7)
- net PB10: now also J4.15 (Pin_15); no longer J4.6 (Pin_6)
- net PB11: now also J4.16 (Pin_16); no longer J4.5 (Pin_5)
- net PC13: now also J4.2 (Pin_2); no longer J4.19 (Pin_19)
- net PC14: now also J4.3 (Pin_3); no longer J4.18 (Pin_18)
- net PC15: now also J4.4 (Pin_4); no longer J4.17 (Pin_17)
- net VBUS: now also C14.1
Changed lines of the file:
@@
 L Connector_Generic:Conn_01x20 J4
 U 1 1 5DEFA97C
-P 10800 5250
-F 0 "J4" H 10750 6350 50  0000 L CNN
-F 1 "Right Castellation" H 10450 6300 50  0001 L CNN
-F 2 "Connector_PinHeader_2.54mm:PinHeader_1x20_P2.54mm_Vertical" H 10800 5250 50  0001 C CNN
-F 3 "~" H 10800 5250 50  0001 C CNN
-	1    10800 5250
-	1    0    0    -1
+P 10800 5350
+F 0 "J4" H 10750 6450 50  0000 L CNN
+F 1 "Right Castellation" H 10450 6400 50  0001 L CNN
+F 2 "Connector_PinHeader_2.54mm:PinHeader_1x20_P2.54mm_Vertical" H 10800 5350 50  0001 C CNN
+F 3 "~" H 10800 5350 50  0001 C CNN
+	1    10800 5350
+	1    0    0    1
 $EndComp
 Text Notes 10750 4150 2    100  Italic 20
@@
 	10550 4450 10550 4350
 Wire Wire Line
-	10550 4250 11000 4250
+	10550 4250 10600 4250
 Wire Wire Line
 	11000 4250 11000 4450
@@
 Wire Wire Line
 	9250 3000 9400 3000
+$Comp
+L power:VBUS #PWR042
+U 1 1 5E28CF9E
+P 750 3100
+F 0 "#PWR042" H 750 2950 50  0001 C CNN
+F 1 "VBUS" H 765 3273 50  0000 C CNN
+F 2 "" H 750 3100 50  0001 C CNN
+F 3 "" H 750 3100 50  0001 C CNN
+	1    750  3100
+	1    0    0    -1
+$EndComp
+$Comp
+L Device:C C14
+U 1 1 5E28D22C
+P 750 3250
+F 0 "C14" H 865 3296 50  0000 L CNN
+F 1 "100n" H 865 3205 50  0000 L CNN
+F 2 "Capacitor_SMD:C_0603_1608Metric_Pad1.05x0.95mm_HandSolder" H 788 3100 50  0001 C CNN
+F 3 "~" H 750 3250 50  0001 C CNN
+	1    750  3250
+	1    0    0    -1
+$EndComp
+$Comp
+L power:GNDREF #PWR043
+U 1 1 5E28DB6A
+P 750 3400
+F 0 "#PWR043" H 750 3150 50  0001 C CNN
+F 1 "GNDREF" H 755 3227 50  0000 C CNN
+F 2 "" H 750 3400 50  0001 C CNN
+F 3 "" H 750 3400 50  0001 C CNN
+	1    750  3400
+	1    0    0    -1
+$EndComp
+Connection ~ 10600 4250
+Wire Wire Line
+	10600 4250 11000 4250
 $EndSCHEMATC

Commit message: minor updates
Parts:
- added F1: 1A, Fuse:Fuse_0805_2012Metric, symbol Device:Polyfuse
- D1: value Protection -> 1A
Connections:
- net VBUS: now also F1.2; no longer D1.2 (A)
- new net: D1.2 (A), F1.1
Other:
- moved on the sheet: D1
Changed lines of the file:
@@
-	1    0    0    -1
-$EndComp
-$Comp
-L power:VBUS #PWR06
-U 1 1 5DED193B
-P 1700 1000
-F 0 "#PWR06" H 1700 850 50  0001 C CNN
-F 1 "VBUS" H 1715 1173 50  0000 C CNN
-F 2 "" H 1700 1000 50  0001 C CNN
-F 3 "" H 1700 1000 50  0001 C CNN
-	1    1700 1000
 	1    0    0    -1
 $EndComp
@@
 Text Notes 2600 700  0    100  Italic 20
 USB to serial (VCP)
-$Comp
-L power:+5V #PWR09
-U 1 1 5E127D96
-P 2300 1000
-F 0 "#PWR09" H 2300 850 50  0001 C CNN
-F 1 "+5V" H 2315 1173 50  0000 C CNN
-F 2 "" H 2300 1000 50  0001 C CNN
-F 3 "" H 2300 1000 50  0001 C CNN
-	1    2300 1000
-	1    0    0    -1
-$EndComp
-$Comp
-L Device:D_Schottky_ALT D1
-U 1 1 5E12857D
-P 2000 1050
-F 0 "D1" H 2000 834 50  0000 C CNN
-F 1 "Protection" H 2000 925 50  0000 C CNN
-F 2 "Diode_SMD:D_SOD-128" H 2000 1050 50  0001 C CNN
-F 3 "~" H 2000 1050 50  0001 C CNN
-	1    2000 1050
-	-1   0    0    1
-$EndComp
-Wire Wire Line
-	2150 1050 2300 1050
-Wire Wire Line
-	1600 1050 1700 1050
-Wire Wire Line
-	1700 1000 1700 1050
-Connection ~ 1700 1050
-Wire Wire Line
-	1700 1050 1850 1050
-Wire Wire Line
-	2300 1000 2300 1050
 Wire Wire Line
 	2850 1550 2800 1550
@@
 	10550 4450 10550 4350
 Wire Wire Line
-	10550 4250 10600 4250
-Wire Wire Line
 	11000 4250 11000 4450
 Wire Wire Line
@@
 	1    0    0    -1
 $EndComp
-Connection ~ 10600 4250
-Wire Wire Line
-	10600 4250 11000 4250
+Wire Wire Line
+	10550 4250 11000 4250
+$Comp
+L power:VBUS #PWR06
+U 1 1 5DED193B
+P 1650 950
+F 0 "#PWR06" H 1650 800 50  0001 C CNN
+F 1 "VBUS" H 1665 1123 50  0000 C CNN
+F 2 "" H 1650 950 50  0001 C CNN
+F 3 "" H 1650 950 50  0001 C CNN
+	1    1650 950
+	1    0    0    -1
+$EndComp
+$Comp
+L Device:Polyfuse F1
+U 1 1 5E2D46C7
+P 1850 1050
+F 0 "F1" V 1625 1050 50  0000 C CNN
+F 1 "1A" V 1716 1050 50  0000 C CNN
+F 2 "Fuse:Fuse_0805_2012Metric" H 1900 850 50  0001 L CNN
+F 3 "~" H 1850 1050 50  0001 C CNN
+	1    1850 1050
+	0    1    1    0
+$EndComp
+$Comp
+L Device:D_Schottky_ALT D1
+U 1 1 5E12857D
+P 2150 1050
+F 0 "D1" H 2150 834 50  0000 C CNN
+F 1 "1A" H 2150 925 50  0000 C CNN
+F 2 "Diode_SMD:D_SOD-128" H 2150 1050 50  0001 C CNN
+F 3 "~" H 2150 1050 50  0001 C CNN
+	1    2150 1050
+	-1   0    0    1
+$EndComp
+$Comp
+L power:+5V #PWR09
+U 1 1 5E127D96
+P 2350 950
+F 0 "#PWR09" H 2350 800 50  0001 C CNN
+F 1 "+5V" H 2365 1123 50  0000 C CNN
+F 2 "" H 2350 950 50  0001 C CNN
+F 3 "" H 2350 950 50  0001 C CNN
+	1    2350 950
+	1    0    0    -1
+$EndComp
+Wire Wire Line
+	2300 1050 2350 1050
+Wire Wire Line
+	2350 1050 2350 950
+Wire Wire Line
+	1700 1050 1650 1050
+Wire Wire Line
+	1650 950  1650 1050
+Connection ~ 1650 1050
+Wire Wire Line
+	1650 1050 1600 1050
 $EndSCHEMATC
